File: IOB-Adapter-Input_array.brd (EAGLE design)
At the start: 106.7 x 104.1 mm, 173 parts

Commit message: added values for connectors
Parts:
- CARRIER: value (none) -> 10x10
- FID-LR, FID-UL: value (none) -> FIDUCIAL
Changed lines of the file:
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@@
 <element name="R11X52" library="SPCoast" package="0805-RES" value="82R" x="85.725" y="75.819" rot="R90"/>
 <element name="R12X52" library="SPCoast" package="0805-RES" value="82R" x="82.296" y="75.819" rot="R90"/>
-<element name="CARRIER" library="SPCoast" package="BOARD-DINRAIL-3.17IN-5X2-IOP" value="" x="0" y="0"/>
-<element name="FID-UL" library="SPCoast" package="FIDUCIAL_1MM" value="" x="5.08" y="91.44" smashed="yes">
+<element name="CARRIER" library="SPCoast" package="BOARD-DINRAIL-3.17IN-5X2-IOP" value="10x10" x="0" y="0"/>
+<element name="FID-UL" library="SPCoast" package="FIDUCIAL_1MM" value="FIDUCIAL" x="5.08" y="91.44" smashed="yes">
 <attribute name="NAME" x="2.54" y="89.535" size="1.016" layer="25" rot="R90"/>
 </element>
-<element name="FID-LR" library="SPCoast" package="FIDUCIAL_1MM" value="" x="93.98" y="10.16" smashed="yes">
+<element name="FID-LR" library="SPCoast" package="FIDUCIAL_1MM" value="FIDUCIAL" x="93.98" y="10.16" smashed="yes">
 <attribute name="NAME" x="99.06" y="6.985" size="1.016" layer="25" rot="R90"/>
 </element>

Commit message: normalized values
Parts:
- CARRIER: value 10x10 -> BOARD
Changed lines of the file:
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@@
 <element name="R11X52" library="SPCoast" package="0805-RES" value="82R" x="85.725" y="75.819" rot="R90"/>
 <element name="R12X52" library="SPCoast" package="0805-RES" value="82R" x="82.296" y="75.819" rot="R90"/>
-<element name="CARRIER" library="SPCoast" package="BOARD-DINRAIL-3.17IN-5X2-IOP" value="10x10" x="0" y="0"/>
+<element name="CARRIER" library="SPCoast" package="BOARD-DINRAIL-3.17IN-5X2-IOP" value="BOARD" x="0" y="0"/>
 <element name="FID-UL" library="SPCoast" package="FIDUCIAL_1MM" value="FIDUCIAL" x="5.08" y="91.44" smashed="yes">
 <attribute name="NAME" x="2.54" y="89.535" size="1.016" layer="25" rot="R90"/>
